Commit message: Get a real URDF model and meshes; remove some cruft
On the original SD card that shipped with Dogzilla is a docker image,
and their tech support told me that it contains a URDF file.
What I found in there instead is
/root/yahboomcar_ws/src/yahboom_description/urdf/yahboom_xgo_rviz_local.xacro
which is a xacro template for a URDF file; and meshes are in various places including
/root/yahboomcar_ws/src/yahboom_description/meshes/XGO
The urdf/dogzilla.urdf here is made by expanding the xacro macros by hand,
because the intended way to do that is not part of the dogzilla tutorials
as far as I can tell. And it seems the Dogzilla is based on the XGO robots,
so apparently the model also was copied from there.

The result is viewable with [urdf-viz](https://github.com/openrr/urdf-viz).
Gazebo still complains so far:

```
$ gz sim dogzilla.urdf
Warning [Utils.cc:115] Non-unique name[lf_lower_leg_link] detected 2 times in XML children of model with name[xgo].[Err] [Server.cc:86] Error Code 2: Msg: Link with name [lf_lower_leg_link] in model with name [xgo] has a name collision. Please rename this link.
[Err] [Server.cc:86] Error Code 2: Msg: Joint with non-unique name [lf_lower_leg_link] detected in model with name [xgo].
[Err] [Server.cc:86] Error Code 25: Msg: FrameAttachedToGraph error, LINK vertex with name [xgo::lf_lower_leg_link] should have no outgoing edges in MODEL attached_to graph.
[Err] [Server.cc:86] Error Code 24: Msg: FrameAttachedToGraph cycle detected, already visited vertex [xgo::lf_lower_leg_link].
[Err] [Server.cc:86] Error Code 2: Msg: Joint with non-unique name [lf_lower_leg_link] detected in model with name [xgo].
[Err] [Server.cc:86] Error Code 27: Msg: relative_to name[lf_lower_leg_link] is identical to link name[lf_lower_leg_link], causing a graph cycle in model with name[xgo].
[Err] [Server.cc:86] Error Code 28: Msg: PoseRelativeToGraph error, too many incoming edges at a vertex with name [xgo::lf_lower_leg_link].
[Err] [Server.cc:86] Error Code 28: Msg: PoseRelativeToGraph error: multiple incoming edges to current vertex [xgo::lf_lower_leg_link].
[Err] [Server.cc:86] Error Code 20: Msg: joint with name[lf_lower_leg_link] in model with name[xgo] must not specify its own name as the child frame.
[Err] [Server.cc:86] Error Code 24: Msg: FrameAttachedToGraph cycle detected, already visited vertex [xgo::lf_lower_leg_link].
[Err] [Server.cc:86] Error Code 28: Msg: PoseRelativeToGraph error: multiple incoming edges to current vertex [xgo::lf_lower_leg_link].
[Err] [Server.cc:86] Error Code 28: Msg: PoseRelativeToGraph error: multiple incoming edges to current vertex [xgo::lf_lower_leg_link].
```

File: dogzilla/urdf/dogzilla.urdf (robot description, URDF)
Before this commit: robot fifi, 0 links, 0 joints
Links:
- added link base_footprint
- added link base_link, mass 0.387351847505872; collision mesh filename=meshes/base_link.STL; visual mesh filename=meshes/base_link.STL
- added link camera_link, mass 0.00465716120355248; collision mesh filename=meshes/camera_link.STL; visual mesh filename=meshes/camera_link.STL
- added link imu_link, mass 0.0141156733693049; collision mesh filename=meshes/laser_link.STL; visual mesh filename=meshes/laser_link.STL
- added link laser_link, mass 0.0141156733693049; collision mesh filename=meshes/laser_link.STL; visual mesh filename=meshes/laser_link.STL
- added link lf_hip_link, mass 0.019600254805245; collision mesh filename=meshes/lf_hip_link.STL; visual mesh filename=meshes/lf_hip_link.STL
- added link lf_lower_leg_link, mass 0.022687879462132; collision mesh filename=meshes/lf_lower_leg_link.STL; visual mesh filename=meshes/lf_lower_leg_link.STL
- added link lf_upper_leg_link, mass 0.012342949675616; collision mesh filename=meshes/lf_upper_leg_link.STL; visual mesh filename=meshes/lf_upper_leg_link.STL
- added link lh_hip_link, mass 0.019600254805245; collision mesh filename=meshes/lh_hip_link.STL; visual mesh filename=meshes/lh_hip_link.STL
- added link lh_lower_leg_link, mass 0.0226878794439316; collision mesh filename=meshes/lh_lower_leg_link.STL; visual mesh filename=meshes/lh_lower_leg_link.STL
- added link lh_upper_leg_link, mass 0.0123429496756159; collision mesh filename=meshes/lh_upper_leg_link.STL; visual mesh filename=meshes/lh_upper_leg_link.STL
- added link rf_hip_link, mass 0.00980012555956536; collision mesh filename=meshes/rf_hip_link.STL; visual mesh filename=meshes/rf_hip_link.STL
- added link rf_lower_leg_link, mass 0.0226878794123114; collision mesh filename=meshes/rf_lower_leg_link.STL; visual mesh filename=meshes/rf_lower_leg_link.STL
- added link rf_upper_leg_link, mass 0.0123429496756159; collision mesh filename=meshes/rf_upper_leg_link.STL; visual mesh filename=meshes/rf_upper_leg_link.STL
- added link rh_hip_link, mass 0.00980012555956509; collision mesh filename=meshes/rh_hip_link.STL; visual mesh filename=meshes/rh_hip_link.STL
- added link rh_lower_leg_link, mass 0.0226878792028959; collision mesh filename=meshes/rh_lower_leg_link.STL; visual mesh filename=meshes/rh_lower_leg_link.STL
- added link rh_upper_leg_link, mass 0.0123429496756159; collision mesh filename=meshes/rh_upper_leg_link.STL; visual mesh filename=meshes/rh_upper_leg_link.STL
Joints:
- added joint base_joint: type fixed, parent base_footprint, child base_link, origin xyz=0 0 0.010 rpy=0 0 0
- added joint camera_Joint: type fixed, parent base_link, child camera_link, origin xyz=0.075751 0 0.059653 rpy=0 0 0, axis 0 0 0
- added joint imu_Joint: type fixed, parent base_link, child imu_link, origin xyz=0.085 4.4164E-05 0.070 rpy=0 0 0, axis 0 0 0
- added joint laser_Joint: type fixed, parent base_link, child laser_link, origin xyz=-0.016732 4.4164E-05 0.10335 rpy=0 0 0, axis 0 0 0
- added joint lf_hip_joint: type revolute, parent base_link, child lf_hip_link, origin xyz=0.09332 0.022407 0.01454 rpy=0 0 0, axis -1 0 0, limit lower=-3.141592654 upper=3.141592654 effort=25 velocity=1.5
- added joint lf_lower_leg_link: type revolute, parent lf_upper_leg_link, child lf_lower_leg_link, origin xyz=0 -0.00072 -0.059896 rpy=0 0 0, axis 0 1 0, limit lower=-3.141592654 upper=3.141592654 effort=25 velocity=1.5
- added joint lf_upper_leg_joint: type revolute, parent lf_hip_link, child lf_upper_leg_link, origin xyz=-0.018325 0.049313 0 rpy=0 0 0, axis 0 1 0, limit lower=-3.141592654 upper=3.141592654 effort=25 velocity=1.5
- added joint lh_hip_joint: type revolute, parent base_link, child lh_hip_link, origin xyz=-0.05668 0.022407 0.01454 rpy=0 0 0, axis 1 0 0, limit lower=-3.141592654 upper=3.141592654 effort=25 velocity=1.5
- added joint lh_lower_leg_joint: type revolute, parent lh_upper_leg_link, child lh_lower_leg_link, origin xyz=0 -0.00072 -0.059896 rpy=0 0 0, axis 0 1 0, limit lower=-3.141592654 upper=3.141592654 effort=25 velocity=1.5
- added joint lh_upper_leg_joint: type revolute, parent lh_hip_link, child lh_upper_leg_link, origin xyz=-0.0183249999999999 0.0493130541805868 0 rpy=0 0 0, axis 0 1 0, limit lower=-3.141592654 upper=3.141592654 effort=25 velocity=1.5
- added joint rf_hip_joint: type revolute, parent base_link, child rf_hip_link, origin xyz=0.09332 -0.022517 0.01454 rpy=0 0 0, axis -1 0 0, limit lower=-3.141592654 upper=3.141592654 effort=25 velocity=1.5
- added joint rf_lower_leg_joint: type revolute, parent rf_upper_leg_link, child rf_lower_leg_link, origin xyz=0 0 -0.059896 rpy=0 0 0, axis 0 -1 0, limit lower=-3.141592654 upper=3.141592654 effort=25 velocity=1.5
- added joint rf_upper_leg_joint: type revolute, parent rf_hip_link, child rf_upper_leg_link, origin xyz=-0.018325 -0.049313 0 rpy=0 0 0, axis 0 -1 0, limit lower=-3.141592654 upper=3.141592654 effort=25 velocity=1.5
- added joint rh_hip_joint: type revolute, parent base_link, child rh_hip_link, origin xyz=-0.05668 -0.022517 0.01454 rpy=0 0 0, axis 1 0 0, limit lower=-3.141592654 upper=3.141592654 effort=25 velocity=1.5
- added joint rh_lower_leg_joint: type revolute, parent rh_upper_leg_link, child rh_lower_leg_link, origin xyz=0 0 -0.059896 rpy=0 0 0, axis 0 -1 0, limit lower=-3.141592654 upper=3.141592654 effort=25 velocity=1.5
- added joint rh_upper_leg_joint: type revolute, parent rh_hip_link, child rh_upper_leg_link, origin xyz=-0.018325 -0.049313 0 rpy=0 0 0, axis 0 -1 0, limit lower=-3.141592654 upper=3.141592654 effort=25 velocity=1.5

Commit message: Rename a couple of things in dogzilla.urdf: satisfy gazebo
The complaint was because a joint should not have the same name
as a link.

File: dogzilla/urdf/dogzilla.urdf (robot description, URDF)
Before this commit: robot xgo, 17 links, 16 joints
Joints:
- removed joint lf_lower_leg_link
- added joint lf_lower_leg_joint: type revolute, parent lf_upper_leg_link, child lf_lower_leg_link, origin xyz=0 -0.00072 -0.059896 rpy=0 0 0, axis 0 1 0, limit lower=-3.141592654 upper=3.141592654 effort=25 velocity=1.5

Commit message: Replace STL file for "imu_link" with a box resembling an internal PCB
I'm not exactly sure where the IMU chip is, but it's certainly not
a second LiDAR sticking up from the dog's nose.

File: dogzilla/urdf/dogzilla.urdf (robot description, URDF)
Before this commit: robot dogzilla, 17 links, 16 joints
Links:
- link imu_link: geometry collision mesh filename=meshes/laser_link.STL; visual box size=0.02 0.020 0.001

Commit message: Try to fix the joint ranges of motion
It was allowing impossible poses. Fix the URDF first, then redo the
code generation, and keep only the relevant changes.

However, there is some asymmetry: for example if we drag sliders to set
the RhUpperLegLink and LhUpperLegLink angles to the most-positive values,
one swings forward and one swings backward.

File: dogzilla/urdf/dogzilla.urdf (robot description, URDF)
Before this commit: robot dogzilla, 17 links, 16 joints
Joints:
- joint lf_hip_joint: limit lower=-3.141592654 upper=3.141592654 effort=25 velocity=1.5 -> lower=-0.541052068 upper=0.541052068 effort=25 velocity=1.5
- joint lf_lower_leg_joint: limit lower=-3.141592654 upper=3.141592654 effort=25 velocity=1.5 -> lower=-3.054326191 upper=-0.9948376737 effort=25 velocity=1.5
- joint lf_upper_leg_joint: limit lower=-3.141592654 upper=3.141592654 effort=25 velocity=1.5 -> lower=-1.151917306 upper=1.623156204 effort=25 velocity=1.5
- joint lh_hip_joint: limit lower=-3.141592654 upper=3.141592654 effort=25 velocity=1.5 -> lower=-0.541052068 upper=0.541052068 effort=25 velocity=1.5
- joint lh_lower_leg_joint: limit lower=-3.141592654 upper=3.141592654 effort=25 velocity=1.5 -> lower=-3.054326191 upper=-0.9948376737 effort=25 velocity=1.5
- joint lh_upper_leg_joint: limit lower=-3.141592654 upper=3.141592654 effort=25 velocity=1.5 -> lower=-1.151917306 upper=1.623156204 effort=25 velocity=1.5
- joint rf_hip_joint: limit lower=-3.141592654 upper=3.141592654 effort=25 velocity=1.5 -> lower=-0.541052068 upper=0.541052068 effort=25 velocity=1.5
- joint rf_lower_leg_joint: limit lower=-3.141592654 upper=3.141592654 effort=25 velocity=1.5 -> lower=-3.054326191 upper=-0.9948376737 effort=25 velocity=1.5
- joint rf_upper_leg_joint: limit lower=-3.141592654 upper=3.141592654 effort=25 velocity=1.5 -> lower=-1.151917306 upper=1.623156204 effort=25 velocity=1.5
- joint rh_hip_joint: limit lower=-3.141592654 upper=3.141592654 effort=25 velocity=1.5 -> lower=-0.541052068 upper=0.541052068 effort=25 velocity=1.5
- joint rh_lower_leg_joint: limit lower=-3.141592654 upper=3.141592654 effort=25 velocity=1.5 -> lower=-3.054326191 upper=-0.9948376737 effort=25 velocity=1.5
- joint rh_upper_leg_joint: limit lower=-3.141592654 upper=3.141592654 effort=25 velocity=1.5 -> lower=-1.151917306 upper=1.623156204 effort=25 velocity=1.5

Commit message: Fix the joint ranges of motion
Some axes needed reversing. Now I think the URDF-specified ranges
should match the motor controller's ranges and directions:
to fold the lower leg up to the thigh is the most-negative angle;
to fold the upper leg up to the body is the most-positive angle;
to angle a hip joint outwards away from the body is most-positive.

File: dogzilla/urdf/dogzilla.urdf (robot description, URDF)
Before this commit: robot dogzilla, 17 links, 16 joints
Joints:
- joint lf_hip_joint: axis -1 0 0 -> 1 0 0
- joint rf_lower_leg_joint: axis 0 -1 0 -> 0 1 0
- joint rf_upper_leg_joint: axis 0 -1 0 -> 0 1 0
- joint rh_hip_joint: axis 1 0 0 -> -1 0 0
- joint rh_lower_leg_joint: axis 0 -1 0 -> 0 1 0
- joint rh_upper_leg_joint: axis 0 -1 0 -> 0 1 0

Commit message: Fix up the lower leg range of motion again
The motor controller range is
- lower leg folded almost up to thigh: -73
- lower leg at 90 degrees to thigh: 16 (as measured)
- lower leg fully extended: 57

So it's "off by" 106 degrees from the angular range as we render it.
(Since the motor controller uses signed 8-bit values, the zero value had
to be something reasonable, I suppose.) This correction makes it
look correct in the "digital twin".

Amends 063db7bdb446401027c3224a7b4945aa1960577b : the lower limit
(lower leg fully extended) is -43 (90 - 57), not -57.

File: dogzilla/urdf/dogzilla.urdf (robot description, URDF)
Before this commit: robot dogzilla, 17 links, 16 joints
Joints:
- joint lf_lower_leg_joint: limit lower=-3.054326191 upper=-0.9948376737 effort=25 velocity=1.5 -> lower=-3.054326191 upper=-0.750491578455556 effort=25 velocity=1.5
- joint lh_lower_leg_joint: limit lower=-3.054326191 upper=-0.9948376737 effort=25 velocity=1.5 -> lower=-3.054326191 upper=-0.750491578455556 effort=25 velocity=1.5
- joint rf_lower_leg_joint: limit lower=-3.054326191 upper=-0.9948376737 effort=25 velocity=1.5 -> lower=-3.054326191 upper=-0.750491578455556 effort=25 velocity=1.5
- joint rh_lower_leg_joint: limit lower=-3.054326191 upper=-0.9948376737 effort=25 velocity=1.5 -> lower=-3.054326191 upper=-0.750491578455556 effort=25 velocity=1.5
